File: HS_Pair_Test/simple/simple.sch (KiCad schematic (older format))
At the start: 3 parts, among them P101 CONN_01X02, P102 CONN_01X02, P103 CONN_01X02

Commit message: changed the simple example with a SMT connector
Parts:
- P101, P102: footprint Connectors_254mm:pin_array_2x1 -> test:TEST_01x02_05mm
Changed lines of the file:
@@
 LIBS:contrib
 LIBS:valves
+LIBS:simple-cache
 EELAYER 25 0
 EELAYER END
@@
 F 0 "P102" H 8100 3300 50  0000 C CNN
 F 1 "CONN_01X02" V 8200 3150 50  0000 C CNN
-F 2 "Connectors_254mm:pin_array_2x1" H 8100 3150 60  0001 C CNN
+F 2 "test:TEST_01x02_05mm" H 8100 3150 60  0001 C CNN
 F 3 "" H 8100 3150 60  0000 C CNN
 	1    8100 3150
@@
 F 0 "P101" H 5575 3300 50  0000 C CNN
 F 1 "CONN_01X02" V 5675 3150 50  0000 C CNN
-F 2 "Connectors_254mm:pin_array_2x1" H 5575 3150 60  0001 C CNN
+F 2 "test:TEST_01x02_05mm" H 5575 3150 60  0001 C CNN
 F 3 "" H 5575 3150 60  0000 C CNN
 	1    5575 3150
