File: meta_tester/board/si5338.sch (KiCad schematic (older format))
At the start: 24 parts, among them U701 Si5338, X701 25MHz

Commit message: starting layout
Parts:
- C701: footprint SM0805 -> General_SMD:SM0805
- C702, C703, C704, C705, C706, C707, C708, C709, C710, C711, C712, C713, C714, C715, R701, R702, R703, R704, R705, R706, R707: footprint SM0402 -> General_SMD:SM0402
Changed lines of the file:
@@
 EESchema Schematic File Version 2
+LIBS:meta_tester_si5338-rescue
 LIBS:power
 LIBS:device
@@
 LIBS:tca0372
 LIBS:MAX571X-TSSOP14
+LIBS:EFM32
+LIBS:stm32f103tb-qfn36
+LIBS:ch340
+LIBS:reg113-xx-sot23
+LIBS:RF_Connectors
+LIBS:antenna
 LIBS:meta_tester_si5338-cache
 EELAYER 25 0
@@
 $EndComp
 $Comp
-L GND #PWR0124
+L GND #PWR048
 U 1 1 5718D4E9
 P 5525 4300
-F 0 "#PWR0124" H 5525 4050 50  0001 C CNN
+F 0 "#PWR048" H 5525 4050 50  0001 C CNN
 F 1 "GND" H 5525 4150 50  0001 C CNN
 F 2 "" H 5525 4300 50  0000 C CNN
@@
 F 0 "C701" H 2550 5000 25  0000 C CNN
 F 1 "10uF" H 2550 5175 25  0000 C CNN
-F 2 "SM0805" H 2550 5200 60  0001 C CNN
+F 2 "General_SMD:SM0805" H 2550 5200 60  0001 C CNN
 F 3 "" H 2550 5100 60  0000 C CNN
 	1    2550 5100
@@
 $EndComp
 $Comp
-L GND #PWR0125
+L GND #PWR049
 U 1 1 5718D63A
 P 2550 5300
-F 0 "#PWR0125" H 2550 5050 50  0001 C CNN
+F 0 "#PWR049" H 2550 5050 50  0001 C CNN
 F 1 "GND" H 2550 5150 50  0001 C CNN
 F 2 "" H 2550 5300 50  0000 C CNN
@@
 F 0 "C702" H 2775 5000 25  0000 C CNN
 F 1 "0.1u" H 2775 5175 25  0000 C CNN
-F 2 "SM0402" H 2775 5200 60  0001 C CNN
+F 2 "General_SMD:SM0402" H 2775 5200 60  0001 C CNN
 F 3 "" H 2775 5100 60  0000 C CNN
 	1    2775 5100
@@
 F 0 "C703" H 3000 5000 25  0000 C CNN
 F 1 "0.1u" H 3000 5175 25  0000 C CNN
-F 2 "SM0402" H 3000 5200 60  0001 C CNN
+F 2 "General_SMD:SM0402" H 3000 5200 60  0001 C CNN
 F 3 "" H 3000 5100 60  0000 C CNN
 	1    3000 5100
@@
 	4525 3750 5400 3750
 $Comp
-L GND #PWR0126
+L GND #PWR050
 U 1 1 57189ECB
 P 4150 3950
-F 0 "#PWR0126" H 4150 3700 50  0001 C CNN
+F 0 "#PWR050" H 4150 3700 50  0001 C CNN
 F 1 "GND" H 4150 3800 50  0001 C CNN
 F 2 "" H 4150 3950 50  0000 C CNN
@@
 	4150 3825 4150 3950
 $Comp
-L GND #PWR0127
+L GND #PWR051
 U 1 1 57189F40
 P 4400 3650
-F 0 "#PWR0127" H 4400 3400 50  0001 C CNN
+F 0 "#PWR051" H 4400 3400 50  0001 C CNN
 F 1 "GND" H 4400 3500 50  0001 C CNN
 F 2 "" H 4400 3650 50  0000 C CNN
@@
 F 0 "R701" H 4600 2275 25  0000 C CNN
 F 1 "10k" H 4600 2425 25  0000 C CNN
-F 2 "SM0402" H 4600 2375 60  0001 C CNN
+F 2 "General_SMD:SM0402" H 4600 2375 60  0001 C CNN
 F 3 "" H 4600 2375 60  0000 C CNN
 	1    4600 2375
@@
 F 0 "R702" H 4825 2275 25  0000 C CNN
 F 1 "10k" H 4825 2425 25  0000 C CNN
-F 2 "SM0402" H 4825 2375 60  0001 C CNN
+F 2 "General_SMD:SM0402" H 4825 2375 60  0001 C CNN
 F 3 "" H 4825 2375 60  0000 C CNN
 	1    4825 2375
@@
 F 0 "C704" H 3250 5000 25  0000 C CNN
 F 1 "0.1u" H 3250 5175 25  0000 C CNN
-F 2 "SM0402" H 3250 5200 60  0001 C CNN
+F 2 "General_SMD:SM0402" H 3250 5200 60  0001 C CNN
 F 3 "" H 3250 5100 60  0000 C CNN
 	1    3250 5100
@@
 F 0 "C705" H 3500 5000 25  0000 C CNN
 F 1 "0.1u" H 3500 5175 25  0000 C CNN
-F 2 "SM0402" H 3500 5200 60  0001 C CNN
+F 2 "General_SMD:SM0402" H 3500 5200 60  0001 C CNN
 F 3 "" H 3500 5100 60  0000 C CNN
 	1    3500 5100
@@
 F 0 "C706" H 3750 5000 25  0000 C CNN
 F 1 "0.1u" H 3750 5175 25  0000 C CNN
-F 2 "SM0402" H 3750 5200 60  0001 C CNN
+F 2 "General_SMD:SM0402" H 3750 5200 60  0001 C CNN
 F 3 "" H 3750 5100 60  0000 C CNN
 	1    3750 5100
@@
 F 0 "C707" H 4025 5000 25  0000 C CNN
 F 1 "0.1u" H 4025 5175 25  0000 C CNN
-F 2 "SM0402" H 4025 5200 60  0001 C CNN
+F 2 "General_SMD:SM0402" H 4025 5200 60  0001 C CNN
 F 3 "" H 4025 5100 60  0000 C CNN
 	1    4025 5100
@@
 Connection ~ 3750 4950
 $Comp
-L GND #PWR0128
+L GND #PWR052
 U 1 1 57195D64
 P 5200 4350
-F 0 "#PWR0128" H 5200 4100 50  0001 C CNN
+F 0 "#PWR052" H 5200 4100 50  0001 C CNN
 F 1 "GND" H 5200 4200 50  0001 C CNN
 F 2 "" H 5200 4350 50  0000 C CNN
@@
 F 0 "R703" H 5300 4550 25  0000 C CNN
 F 1 "4.7k" H 5300 4700 25  0000 C CNN
-F 2 "SM0402" H 5300 4650 60  0001 C CNN
+F 2 "General_SMD:SM0402" H 5300 4650 60  0001 C CNN
 F 3 "" H 5300 4650 60  0000 C CNN
 	1    5300 4650
@@
 Connection ~ 5300 4800
 $Comp
-L GND #PWR0129
+L GND #PWR053
 U 1 1 57196D95
 P 5675 3050
-F 0 "#PWR0129" H 5675 2800 50  0001 C CNN
+F 0 "#PWR053" H 5675 2800 50  0001 C CNN
 F 1 "GND" H 5675 2900 50  0001 C CNN
 F 2 "" H 5675 3050 50  0000 C CNN
@@
 F 0 "R705" H 6700 3525 25  0000 C CNN
 F 1 "100" H 6700 3675 25  0000 C CNN
-F 2 "SM0402" H 6700 3625 60  0001 C CNN
+F 2 "General_SMD:SM0402" H 6700 3625 60  0001 C CNN
 F 3 "" H 6700 3625 60  0000 C CNN
 	1    6700 3625
@@
 F 0 "R706" H 6700 4025 25  0000 C CNN
 F 1 "100" H 6700 4175 25  0000 C CNN
-F 2 "SM0402" H 6700 4125 60  0001 C CNN
+F 2 "General_SMD:SM0402" H 6700 4125 60  0001 C CNN
 F 3 "" H 6700 4125 60  0000 C CNN
 	1    6700 4125
@@
 F 0 "R707" H 6700 4625 25  0000 C CNN
 F 1 "100" H 6700 4775 25  0000 C CNN
-F 2 "SM0402" H 6700 4725 60  0001 C CNN
+F 2 "General_SMD:SM0402" H 6700 4725 60  0001 C CNN
 F 3 "" H 6700 4725 60  0000 C CNN
 	1    6700 4725
@@
 F 0 "R704" H 6700 3000 25  0000 C CNN
 F 1 "100" H 6700 3150 25  0000 C CNN
-F 2 "SM0402" H 6700 3100 60  0001 C CNN
+F 2 "General_SMD:SM0402" H 6700 3100 60  0001 C CNN
 F 3 "" H 6700 3100 60  0000 C CNN
 	1    6700 3100
@@
 F 0 "C708" H 7150 2850 25  0000 C CNN
 F 1 "0.1u" H 7150 3025 25  0000 C CNN
-F 2 "SM0402" H 7150 3050 60  0001 C CNN
+F 2 "General_SMD:SM0402" H 7150 3050 60  0001 C CNN
 F 3 "" H 7150 2950 60  0000 C CNN
 	1    7150 2950
@@
 F 0 "C709" H 7150 3175 25  0000 C CNN
 F 1 "0.1u" H 7150 3350 25  0000 C CNN
-F 2 "SM0402" H 7150 3375 60  0001 C CNN
+F 2 "General_SMD:SM0402" H 7150 3375 60  0001 C CNN
 F 3 "" H 7150 3275 60  0000 C CNN
 	1    7150 3275
@@
 F 0 "C710" H 7150 3375 25  0000 C CNN
 F 1 "0.1u" H 7150 3550 25  0000 C CNN
-F 2 "SM0402" H 7150 3575 60  0001 C CNN
+F 2 "General_SMD:SM0402" H 7150 3575 60  0001 C CNN
 F 3 "" H 7150 3475 60  0000 C CNN
 	1    7150 3475
@@
 F 0 "C711" H 7150 3700 25  0000 C CNN
 F 1 "0.1u" H 7150 3875 25  0000 C CNN
-F 2 "SM0402" H 7150 3900 60  0001 C CNN
+F 2 "General_SMD:SM0402" H 7150 3900 60  0001 C CNN
 F 3 "" H 7150 3800 60  0000 C CNN
 	1    7150 3800
@@
 F 0 "C712" H 7150 3850 25  0000 C CNN
 F 1 "0.1u" H 7150 4025 25  0000 C CNN
-F 2 "SM0402" H 7150 4050 60  0001 C CNN
+F 2 "General_SMD:SM0402" H 7150 4050 60  0001 C CNN
 F 3 "" H 7150 3950 60  0000 C CNN
 	1    7150 3950
@@
 F 0 "C713" H 7150 4175 25  0000 C CNN
 F 1 "0.1u" H 7150 4350 25  0000 C CNN
-F 2 "SM0402" H 7150 4375 60  0001 C CNN
+F 2 "General_SMD:SM0402" H 7150 4375 60  0001 C CNN
 F 3 "" H 7150 4275 60  0000 C CNN
 	1    7150 4275
@@
 F 0 "C714" H 7150 4475 25  0000 C CNN
 F 1 "0.1u" H 7150 4650 25  0000 C CNN
-F 2 "SM0402" H 7150 4675 60  0001 C CNN
+F 2 "General_SMD:SM0402" H 7150 4675 60  0001 C CNN
 F 3 "" H 7150 4575 60  0000 C CNN
 	1    7150 4575
@@
 F 0 "C715" H 7150 4775 25  0000 C CNN
 F 1 "0.1u" H 7150 4950 25  0000 C CNN
-F 2 "SM0402" H 7150 4975 60  0001 C CNN
+F 2 "General_SMD:SM0402" H 7150 4975 60  0001 C CNN
 F 3 "" H 7150 4875 60  0000 C CNN
 	1    7150 4875
@@
 clk3_1_N
 $Comp
-L +3.3V #PWR?
+L +3.3V #PWR054
 U 1 1 58AB6DFA
 P 4725 2100
-F 0 "#PWR?" H 4725 1950 50  0001 C CNN
+F 0 "#PWR054" H 4725 1950 50  0001 C CNN
 F 1 "+3.3V" H 4725 2240 50  0000 C CNN
 F 2 "" H 4725 2100 50  0000 C CNN
@@
 $EndComp
 $Comp
-L +3.3V #PWR?
+L +3.3V #PWR055
 U 1 1 58AB7E21
 P 5625 3275
-F 0 "#PWR?" H 5625 3125 50  0001 C CNN
+F 0 "#PWR055" H 5625 3125 50  0001 C CNN
 F 1 "+3.3V" H 5625 3415 50  0000 C CNN
 F 2 "" H 5625 3275 50  0000 C CNN
@@
 $EndComp
 $Comp
-L +3.3V #PWR?
+L +3.3V #PWR056
 U 1 1 58AB850E
 P 5625 4550
-F 0 "#PWR?" H 5625 4400 50  0001 C CNN
+F 0 "#PWR056" H 5625 4400 50  0001 C CNN
 F 1 "+3.3V" H 5625 4690 50  0000 C CNN
 F 2 "" H 5625 4550 50  0000 C CNN
@@
 $EndComp
 $Comp
-L +3.3V #PWR?
+L +3.3V #PWR057
 U 1 1 58ABA203
 P 2550 4900
-F 0 "#PWR?" H 2550 4750 50  0001 C CNN
+F 0 "#PWR057" H 2550 4750 50  0001 C CNN
 F 1 "+3.3V" H 2550 5040 50  0000 C CNN
 F 2 "" H 2550 4900 50  0000 C CNN
