File: meta_tester/board/meta_tester_si5338.kicad_pcb (KiCad board)
At the start: 4 copper layers, 59 x 40 mm, 91 parts, among them J101 SMA_PCB, J102 SMA_PCB, J103 SMA_PCB, J104 SMA_PCB, J105 SMA_PCB, J106 SMA_PCB, J107 SMA_PCB, J108 SMA_PCB, P101 USB_OTG, P102 CONN_01X06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

Commit message: almost finished pcb
Parts:
- C110, R101, R103, R104: moved to F.Cu
- J101, J102, J103, J104, J105, J106, J107, J108: footprint Connectors_RF:Border_Antenna -> Connectors_RF:SMA_AMP_132322
- moved C112 11.6 mm to (164.8, 110.8), turned to 0 degrees
- moved C109 11.0 mm to (162.0, 99.0), turned to 180 degrees
- moved C106 10.3 mm to (164.5, 112.2), turned to 0 degrees
- moved C104 8.93 mm to (161.5, 120.5), turned to 180 degrees
- moved J103 8.41 mm to (197.6, 91.8), turned to 270 degrees
- moved C710 8.27 mm to (191.5, 91.8)
- moved C105 7.55 mm to (162.2, 122.8)
- moved R104 7.55 mm to (164.5, 109.2)
- moved C108 6.61 mm to (161.7, 114.8)
- moved R101 6.37 mm to (161.5, 119.2), turned to 180 degrees
- moved C110 5.44 mm to (161.8, 101.8), turned to 180 degrees
- moved C111 5.39 mm to (162.5, 106.7), turned to 90 degrees
- moved R103 5.26 mm to (162.0, 100.2), turned to 180 degrees
- moved J104 4.32 mm to (197.6, 101.0), turned to 270 degrees
- moved C711 4.03 mm to (191.5, 101.0)
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Connections:
- U102 pad 10: /VddO1 -> /VddO2
- U102 pad 16: /VddO1 -> /VddO2
- U102 pad 2: /VddO0 -> /VddO3
- U102 pad 7: /VddO0 -> /VddO3
- U102 pad 8: /DAC0 -> /DAC1
- U102 pad 9: /DAC1 -> /DAC0
- U103 pad 13: Net-(U103-Pad13) -> /5338_INT
- U104 pad 10: /VddO3 -> /VddO0
- U104 pad 16: /VddO3 -> /VddO0
- U104 pad 2: /VddO2 -> /VddO1
- U104 pad 7: /VddO2 -> /VddO1
- U104 pad 8: /DAC3 -> /DAC2
- U104 pad 9: /DAC2 -> /DAC3
Routing:
- net GND: track 0.00 -> 87.1 mm, vias 0 -> 71
- net +3V3: track 3.94 -> 49.2 mm, vias 0 -> 15
- net /VddO2: track 9.62 -> 35.3 mm, vias 0 -> 2
- net /VddO1: track 11.3 -> 34.9 mm, vias 0 -> 2
- net Net-(R107-Pad1): track 0.00 -> 19.7 mm, vias 0 -> 2
- net Net-(R106-Pad1): track 0.00 -> 18.8 mm, vias 0 -> 2
- net /VddO0: track 9.62 -> 23.8 mm, vias 0 -> 2
- net /VddO3: track 10.9 -> 24.7 mm, vias 0 -> 2
- net /DAC2: track 0.00 -> 12.3 mm
- net Net-(R105-Pad1): track 0.00 -> 9.79 mm, vias 0 -> 2
- net /DAC0: track 0.00 -> 9.07 mm
- net /SI5338/clk1_1_P: track 9.84 -> 16.8 mm
- net +5V: track 0.00 -> 6.68 mm, vias 0 -> 6
- net /SI5338/clk1_1_N: track 9.84 -> 16.3 mm
- net /DAC1: track 0.00 -> 6.33 mm, vias 0 -> 1
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- added copper zone on In2.Cu, net +3V3
- added copper zone on B.Cu, net +5V
- added copper zone on In2.Cu, net +5V
- added copper zone on F.Cu, net /DAC0
- added copper zone on F.Cu, net /DAC1
- added copper zone on F.Cu, net /DAC2
- added copper zone on F.Cu, net /DAC3
- added copper zone on F.Cu, net /PSU01
- added copper zone on B.Cu, net /VddO0
- added copper zone on B.Cu, net /VddO1
- added copper zone on B.Cu, net /VddO2
- added copper zone on B.Cu, net /VddO3
- added copper zone on B.Cu, net GND
- added copper zone on F.Cu, net GND
- added copper zone on In1.Cu, net GND
