File: meta_tester/board/meta_tester_si5338.kicad_pcb (KiCad board)
At the start: 4 copper layers, 59 x 40 mm, 91 parts, among them J101 SMA_PCB, J102 SMA_PCB, J103 SMA_PCB, J104 SMA_PCB, J105 SMA_PCB, J106 SMA_PCB, J107 SMA_PCB, J108 SMA_PCB, P101 USB_OTG, P102 CONN_01X06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

Commit message: finished pcb
Parts:
- added REF**: 2.5mm_non_plated, Mounting_Holes:2.5mm_non_plated, F.Cu at (169.6, 87.0)
- added REF**: 2.5mm_non_plated, Mounting_Holes:2.5mm_non_plated, F.Cu at (143.6, 87.0)
Routing:
- net /SCL: track 1.22 -> 47.4 mm, vias 0 -> 2
- net /SDA: track 1.22 -> 46.7 mm, vias 0 -> 2
- net /5338_INT: track 2.33 -> 37.7 mm, vias 0 -> 2
- net GND: track 87.1 -> 119.7 mm, vias 71 -> 98

Commit message: save before generating gerber
Parts:
- added G***: LOGO, Img:malinois, B.Cu at (158.0, 99.0)
Connections:
- P101 pad 6: GND -> Net-(P101-Pad6)
Routing:
- net GND: track 119.7 -> 259.2 mm, vias 98 -> 160
- net Net-(P101-Pad6): track 0.00 -> 21.5 mm
- net Net-(D101-PadA): track 0.00 -> 1.51 mm
Other:
- board text added: "OpenFPGA Meta Tester nats` nats@more-magic.org"
