File: meta_tester/board/meta_tester_si5338.sch (KiCad schematic (older format))
At the start: 67 parts, among them J101 SMA_PCB, J102 SMA_PCB, J103 SMA_PCB, J104 SMA_PCB, J105 SMA_PCB, J106 SMA_PCB, J107 SMA_PCB, J108 SMA_PCB, P101 USB_OTG, P102 CONN_01X06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

Commit message: save before generating gerber
Connections:
- net GND: no longer P101.6 (shield)
Changed lines of the file:
@@
 	5925 1550 5300 1550
-$Comp
-L GND #PWR015
-U 1 1 58AF1025
-P 8925 1925
-F 0 "#PWR015" H 8925 1675 50  0001 C CNN
-F 1 "GND" H 8925 1775 50  0001 C CNN
-F 2 "" H 8925 1925 50  0000 C CNN
-F 3 "" H 8925 1925 50  0000 C CNN
-	1    8925 1925
-	1    0    0    -1
-$EndComp
 $Comp
 L GND #PWR016
@@
 $EndComp
 Wire Wire Line
-	8925 1850 8925 1925
-Wire Wire Line
 	8525 1650 8425 1650
