File: LabClock/labclock.sch (KiCad schematic (older format))
At the start: 74 parts, among them J101 BNC, J102 BNC, J103 BNC, J104 BNC, J105 USB_OTG, J106 BNC, Q101 BSS138, U101 LT1461AIS8-4, U102 SN74LV4T125, U103 ADF4001_TSSOP16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

Commit message: fixed stuff
Parts:
- C130: value CAP_0402 -> 922pF
- C131: value CAP_0402 -> 6.04nF
- R109: value RES_0402 -> 72.4k
Other:
- note added: "BW: 1kHz\nKv: 40Hz/V\nPFD: 5MHz"
Changed lines of the file:
@@
 P 6100 6125
 F 0 "C130" H 6100 6025 25  0000 C CNN
-F 1 "CAP_0402" H 6100 6200 25  0000 C CNN
+F 1 "922pF" H 6100 6200 25  0000 C CNN
 F 2 "SM0402" H 6100 6225 60  0001 C CNN
 F 3 "" H 6100 6125 60  0000 C CNN
@@
 P 6450 6125
 F 0 "R109" H 6450 6025 25  0000 C CNN
-F 1 "RES_0402" H 6450 6175 25  0000 C CNN
+F 1 "72.4k" H 6450 6175 25  0000 C CNN
 F 2 "SM0402" H 6450 6125 60  0001 C CNN
 F 3 "" H 6450 6125 60  0000 C CNN
@@
 P 6450 6400
 F 0 "C131" H 6450 6300 25  0000 C CNN
-F 1 "CAP_0402" H 6450 6475 25  0000 C CNN
+F 1 "6.04nF" H 6450 6475 25  0000 C CNN
 F 2 "SM0402" H 6450 6500 60  0001 C CNN
 F 3 "" H 6450 6400 60  0000 C CNN
@@
 5V_AMP
 Connection ~ 8350 3125
+Text Notes 6025 5750 0    60   ~ 0
+BW: 1kHz\nKv: 40Hz/V\nPFD: 5MHz
 $EndSCHEMATC
